File: kicad/Bell/Bell.sch (KiCad schematic (older format))
At the start: 9 parts, among them J1 Jack-DC, Q1 Q_NMOS_GDS, U1 NodeMCUv3

Commit message: Kicad: Finished 1st PCB revision
Signed-off-by: CTXz <ctx.xda@gmail.com>
Parts:
- added R2: 100, Resistor_THT:R_Axial_DIN0207_L6.3mm_D2.5mm_P10.16mm_Horizontal, symbol Device:R
- BZ1: footprint (none) -> Buzzer_Beeper:Buzzer_12x9.5RM7.6
- C1: value CP -> 22u; footprint (none) -> Capacitor_THT:CP_Radial_D5.0mm_P2.00mm
- D1: value LED -> Ring LED (5mm WHITE); footprint (none) -> Connector_JST:JST_EH_B2B-EH-A_1x02_P2.50mm_Vertical
- D2: value LED -> Ring LED > 3.3v; footprint (none) -> Connector_JST:JST_EH_B2B-EH-A_1x02_P2.50mm_Vertical
- D3: value LED -> POWER LED (3mm RED); footprint (none) -> Connector_JST:JST_EH_B2B-EH-A_1x02_P2.50mm_Vertical
- J1: footprint (none) -> Connector_JST:JST_EH_B2B-EH-A_1x02_P2.50mm_Vertical
- Q1: footprint (none) -> Package_TO_SOT_THT:TO-220-3_Horizontal_TabDown
- R1: value R -> 10k; footprint (none) -> Resistor_THT:R_Axial_DIN0207_L6.3mm_D2.5mm_P10.16mm_Horizontal
- U1: footprint MODULE_ZC563900 -> ESP8266-Kicad:NodeMCU-LoLinV3
Connections:
- net RING_LED: now also R2.2; no longer D1.2 (A)
- new net: D1.2 (A), R2.1
Other:
- moved on the sheet: D1, D2, Q1
Changed lines of the file:
@@
 F 0 "BZ1" H 4552 1129 50  0000 L CNN
 F 1 "Buzzer" H 4552 1038 50  0000 L CNN
-F 2 "" V 4375 1200 50  0001 C CNN
+F 2 "Buzzer_Beeper:Buzzer_12x9.5RM7.6" V 4375 1200 50  0001 C CNN
 F 3 "~" V 4375 1200 50  0001 C CNN
 	1    4400 1100
@@
 $EndComp
 $Comp
-L Device:LED D2
-U 1 1 61A5B6A0
-P 4400 4100
-F 0 "D2" V 4439 3983 50  0000 R CNN
-F 1 "LED" V 4348 3983 50  0000 R CNN
-F 2 "" H 4400 4100 50  0001 C CNN
-F 3 "~" H 4400 4100 50  0001 C CNN
-	1    4400 4100
-	0    -1   -1   0
-$EndComp
-$Comp
 L Device:Q_NMOS_GDS Q1
 U 1 1 61A5CD90
-P 4300 4600
-F 0 "Q1" H 4504 4646 50  0000 L CNN
-F 1 "Q_NMOS_GDS" H 4504 4555 50  0000 L CNN
-F 2 "" H 4500 4700 50  0001 C CNN
-F 3 "~" H 4300 4600 50  0001 C CNN
-	1    4300 4600
+P 5950 3150
+F 0 "Q1" H 6154 3196 50  0000 L CNN
+F 1 "Q_NMOS_GDS" H 6154 3105 50  0000 L CNN
+F 2 "Package_TO_SOT_THT:TO-220-3_Horizontal_TabDown" H 6150 3250 50  0001 C CNN
+F 3 "~" H 5950 3150 50  0001 C CNN
+	1    5950 3150
 	1    0    0    -1
 $EndComp
@@
 L power:GND #PWR09
 U 1 1 61A5FDFE
-P 4400 4950
-F 0 "#PWR09" H 4400 4700 50  0001 C CNN
-F 1 "GND" H 4405 4777 50  0000 C CNN
-F 2 "" H 4400 4950 50  0001 C CNN
-F 3 "" H 4400 4950 50  0001 C CNN
-	1    4400 4950
-	1    0    0    -1
-$EndComp
-$Comp
-L Device:LED D1
-U 1 1 61A60433
-P 4300 2800
-F 0 "D1" V 4339 2683 50  0000 R CNN
-F 1 "LED" V 4248 2683 50  0000 R CNN
-F 2 "" H 4300 2800 50  0001 C CNN
-F 3 "~" H 4300 2800 50  0001 C CNN
-	1    4300 2800
-	0    -1   -1   0
+P 6050 3500
+F 0 "#PWR09" H 6050 3250 50  0001 C CNN
+F 1 "GND" H 6055 3327 50  0000 C CNN
+F 2 "" H 6050 3500 50  0001 C CNN
+F 3 "" H 6050 3500 50  0001 C CNN
+	1    6050 3500
+	1    0    0    -1
 $EndComp
 $Comp
@@
 U 1 1 61A61407
 P 6350 1000
-F 0 "D3" V 6389 883 50  0000 R CNN
-F 1 "LED" V 6298 883 50  0000 R CNN
-F 2 "" H 6350 1000 50  0001 C CNN
+F 0 "D3" H 6450 850 50  0000 R CNN
+F 1 "POWER LED (3mm RED)" H 6600 1150 25  0000 R CNN
+F 2 "Connector_JST:JST_EH_B2B-EH-A_1x02_P2.50mm_Vertical" H 6350 1000 50  0001 C CNN
 F 3 "~" H 6350 1000 50  0001 C CNN
 	1    6350 1000
@@
 P 5900 1000
 F 0 "R1" V 5693 1000 50  0000 C CNN
-F 1 "R" V 5784 1000 50  0000 C CNN
-F 2 "" V 5830 1000 50  0001 C CNN
+F 1 "10k" V 5784 1000 50  0000 C CNN
+F 2 "Resistor_THT:R_Axial_DIN0207_L6.3mm_D2.5mm_P10.16mm_Horizontal" V 5830 1000 50  0001 C CNN
 F 3 "~" H 5900 1000 50  0001 C CNN
 	1    5900 1000
@@
 F 0 "U1" H 1950 4767 50  0000 C CNN
 F 1 "NodeMCUv3" H 1950 4676 50  0000 C CNN
-F 2 "MODULE_ZC563900" H 1950 3600 50  0001 L BNN
+F 2 "ESP8266-Kicad:NodeMCU-LoLinV3" H 1950 3600 50  0001 L BNN
 F 3 "" H 1950 3600 50  0001 L BNN
 F 4 "N/A" H 1950 3600 50  0001 L BNN "MAXIMUM_PACKAGE_HEIGHT"
@@
 	6650 1000 6500 1000
 Wire Wire Line
-	4400 3800 4400 3950
-Wire Wire Line
-	4400 4250 4400 4400
-Wire Wire Line
-	4400 4800 4400 4950
-Text GLabel 3950 4600 0    50   Input ~ 0
+	6050 2350 6050 2500
+Wire Wire Line
+	6050 2800 6050 2950
+Wire Wire Line
+	6050 3350 6050 3500
+Text GLabel 5600 3150 0    50   Input ~ 0
 RING_LED
 Wire Wire Line
-	3950 4600 4100 4600
+	5600 3150 5750 3150
 $Comp
 L power:VCC #PWR08
 U 1 1 61A82152
-P 4400 3800
-F 0 "#PWR08" H 4400 3650 50  0001 C CNN
-F 1 "VCC" H 4417 3973 50  0000 C CNN
-F 2 "" H 4400 3800 50  0001 C CNN
-F 3 "" H 4400 3800 50  0001 C CNN
-	1    4400 3800
-	1    0    0    -1
-$EndComp
-Text GLabel 4300 2500 1    50   Input ~ 0
+P 6050 2350
+F 0 "#PWR08" H 6050 2200 50  0001 C CNN
+F 1 "VCC" H 6067 2523 50  0000 C CNN
+F 2 "" H 6050 2350 50  0001 C CNN
+F 3 "" H 6050 2350 50  0001 C CNN
+	1    6050 2350
+	1    0    0    -1
+$EndComp
+Text GLabel 4200 2550 1    50   Input ~ 0
 RING_LED
 Wire Wire Line
-	4300 2500 4300 2650
+	4200 2550 4200 2700
 $Comp
 L power:GND #PWR07
 U 1 1 61A8548F
-P 4300 3100
-F 0 "#PWR07" H 4300 2850 50  0001 C CNN
-F 1 "GND" H 4305 2927 50  0000 C CNN
-F 2 "" H 4300 3100 50  0001 C CNN
-F 3 "" H 4300 3100 50  0001 C CNN
-	1    4300 3100
-	1    0    0    -1
-$EndComp
-Wire Wire Line
-	4300 3100 4300 2950
+P 4200 3600
+F 0 "#PWR07" H 4200 3350 50  0001 C CNN
+F 1 "GND" H 4205 3427 50  0000 C CNN
+F 2 "" H 4200 3600 50  0001 C CNN
+F 3 "" H 4200 3600 50  0001 C CNN
+	1    4200 3600
+	1    0    0    -1
+$EndComp
+Wire Wire Line
+	4200 3600 4200 3450
 $Comp
 L Connector:Jack-DC J1
@@
 F 0 "J1" H 957 1525 50  0000 C CNN
 F 1 "Jack-DC" H 957 1434 50  0000 C CNN
-F 2 "" H 950 1160 50  0001 C CNN
+F 2 "Connector_JST:JST_EH_B2B-EH-A_1x02_P2.50mm_Vertical" H 950 1160 50  0001 C CNN
 F 3 "~" H 950 1160 50  0001 C CNN
 	1    900  1200
@@
 P 1850 1400
 F 0 "C1" H 1968 1446 50  0000 L CNN
-F 1 "CP" H 1968 1355 50  0000 L CNN
-F 2 "" H 1888 1250 50  0001 C CNN
+F 1 "22u" H 1968 1355 50  0000 L CNN
+F 2 "Capacitor_THT:CP_Radial_D5.0mm_P2.00mm" H 1888 1250 50  0001 C CNN
 F 3 "~" H 1850 1400 50  0001 C CNN
 	1    1850 1400
@@
 Buzzer
 Wire Notes Line
-	6800 550  6800 1950
-Wire Notes Line
 	550  1950 6800 1950
 Wire Notes Line
@@
 Text Notes 3550 2050 0    50   ~ 0
 Ring Indicator LED - Option 1
-Wire Notes Line
-	5050 550  5050 5300
-Wire Notes Line
-	550  5300 5050 5300
-Wire Notes Line
-	3500 3350 5050 3350
-Text Notes 3550 3450 0    50   ~ 0
+Text Notes 5100 2050 0    50   ~ 0
 Ring Indicator LED - Option 2
+$Comp
+L Device:LED D2
+U 1 1 61A5B6A0
+P 6050 2650
+F 0 "D2" V 6100 2900 50  0000 R CNN
+F 1 "Ring LED > 3.3v" V 6000 3400 50  0000 R CNN
+F 2 "Connector_JST:JST_EH_B2B-EH-A_1x02_P2.50mm_Vertical" H 6050 2650 50  0001 C CNN
+F 3 "~" H 6050 2650 50  0001 C CNN
+	1    6050 2650
+	0    -1   -1   0
+$EndComp
+$Comp
+L Device:R R2
+U 1 1 61D4A297
+P 4200 2850
+F 0 "R2" V 3993 2850 50  0000 C CNN
+F 1 "100" V 4084 2850 50  0000 C CNN
+F 2 "Resistor_THT:R_Axial_DIN0207_L6.3mm_D2.5mm_P10.16mm_Horizontal" V 4130 2850 50  0001 C CNN
+F 3 "~" H 4200 2850 50  0001 C CNN
+	1    4200 2850
+	-1   0    0    1
+$EndComp
+Wire Wire Line
+	4200 3000 4200 3150
+Wire Notes Line
+	3500 3950 6800 3950
+Wire Notes Line
+	6800 550  6800 3950
+Wire Notes Line
+	5050 550  5050 3950
+Wire Notes Line
+	3500 5300 550  5300
+$Comp
+L Device:LED D1
+U 1 1 61A60433
+P 4200 3300
+F 0 "D1" V 4239 3183 50  0000 R CNN
+F 1 "Ring LED (5mm WHITE)" V 4148 3183 39  0000 R CNN
+F 2 "Connector_JST:JST_EH_B2B-EH-A_1x02_P2.50mm_Vertical" H 4200 3300 50  0001 C CNN
+F 3 "~" H 4200 3300 50  0001 C CNN
+	1    4200 3300
+	0    -1   -1   0
+$EndComp
 $EndSCHEMATC
