File: kicad/Bell/Bell.kicad_pcb (KiCad board)
At the start: 2 copper layers, 50.6 x 40.5 mm, 14 parts, among them J1 Jack-DC, Q1 Q_NMOS_GDS, U1 NodeMCUv3

Commit message: Kicad: Updated to v6.0
Signed-off-by: Patrick Pedersen <ctx.xda@gmail.com>
Other:
- net class Default removed
